File: hep-control.sch (KiCad schematic (older format))
At the start: 132 parts, among them U4 Contactor_3phase_2NC_2NO, U6 Contactor_3phase_2NC_2NO, U7 Contactor_3phase_2NC_2NO, U8 Contactor_3phase_2NC_2NO

Commit message: more updoots
Parts:
- gave numbers to parts that had none: 9
Changed lines of the file:
@@
 -24V
 $Comp
-L mrm:Contactor_3phase_2NC_2NO K?
+L mrm:Contactor_3phase_2NC_2NO K20
 U 1 1 5B450ECE
 P 3700 6550
-F 0 "K?" H 3700 6750 50  0000 C CNN
+F 0 "K20" H 3700 6750 50  0000 C CNN
 F 1 "Contactor_3phase_2NC_2NO" H 3700 6350 50  0001 C CNN
 F 2 "" H 4350 6550 50  0001 C CNN
@@
 -24V
 $Comp
-L mrm:Contactor_3phase_2NC_2NO K?
+L mrm:Contactor_3phase_2NC_2NO K21
 U 1 1 5B7FD453
 P 4500 6950
-F 0 "K?" H 4500 7150 50  0000 C CNN
+F 0 "K21" H 4500 7150 50  0000 C CNN
 F 1 "Contactor_3phase_2NC_2NO" H 4500 6750 50  0001 C CNN
 F 2 "" H 5150 6950 50  0001 C CNN
@@
 Connection ~ 9100 6550
 $Comp
-L mrm:Contactor_3phase_2NC_2NO K?
+L mrm:Contactor_3phase_2NC_2NO K16
 U 1 1 5B8C2D32
 P 5400 3750
-F 0 "K?" H 5400 3950 50  0000 C CNN
+F 0 "K16" H 5400 3950 50  0000 C CNN
 F 1 "Contactor_3phase_2NC_2NO" H 5400 3550 50  0001 C CNN
 F 2 "" H 6050 3750 50  0001 C CNN
@@
 $EndComp
 $Comp
-L mrm:Contactor_3phase_2NC_2NO K?
+L mrm:Contactor_3phase_2NC_2NO K17
 U 1 1 5B8C2DC2
 P 7000 3750
-F 0 "K?" H 7000 3950 50  0000 C CNN
+F 0 "K17" H 7000 3950 50  0000 C CNN
 F 1 "Contactor_3phase_2NC_2NO" H 7000 3550 50  0001 C CNN
 F 2 "" H 7650 3750 50  0001 C CNN
@@
 $EndComp
 $Comp
-L mrm:Contactor_3phase_2NC_2NO K?
+L mrm:Contactor_3phase_2NC_2NO K18
 U 1 1 5B8C2E34
 P 9600 3750
-F 0 "K?" H 9600 3950 50  0000 C CNN
+F 0 "K18" H 9600 3950 50  0000 C CNN
 F 1 "Contactor_3phase_2NC_2NO" H 9600 3550 50  0001 C CNN
 F 2 "" H 10250 3750 50  0001 C CNN
@@
 $EndComp
 $Comp
-L mrm:Contactor_3phase_2NC_2NO K?
+L mrm:Contactor_3phase_2NC_2NO K19
 U 1 1 5B8C2EDA
 P 11200 3750
-F 0 "K?" H 11200 3950 50  0000 C CNN
+F 0 "K19" H 11200 3950 50  0000 C CNN
 F 1 "Contactor_3phase_2NC_2NO" H 11200 3550 50  0001 C CNN
 F 2 "" H 11850 3750 50  0001 C CNN
@@
 P 4350 8850
 AR Path="/5AF69061/5BA0BD24" Ref="K?HEP_POWERED?"  Part="6"
-AR Path="/5AE8F11D/5BA0BD24" Ref="K?"  Part="6"
-F 0 "K?" H 4350 8950 50  0000 C CNN
+AR Path="/5AE8F11D/5BA0BD24" Ref="K15"  Part="6"
+F 0 "K15" H 4350 8950 50  0000 C CNN
 F 1 "HEP Voltage Detect" H 4350 8750 50  0000 C CNN
 F 2 "" H 5000 8850 50  0001 C CNN
@@
 -24V
 $Comp
-L mrm:Contactor_3phase_2NC_2NO K?
+L mrm:Contactor_3phase_2NC_2NO K12
 U 5 1 5C040660
 P 3200 2050
-F 0 "K?" H 3200 2300 50  0000 C CNN
+F 0 "K12" H 3200 2300 50  0000 C CNN
 F 1 "Standby Power Selected" H 3200 2200 50  0000 C CNN
 F 2 "" H 3850 2050 50  0001 C CNN
@@
 P 3200 2500
 AR Path="/5AF69061/5C04066B" Ref="K?"  Part="5"
-AR Path="/5AE8F11D/5C04066B" Ref="K?"  Part="5"
-F 0 "K?" H 3200 2750 50  0000 C CNN
+AR Path="/5AE8F11D/5C04066B" Ref="K11"  Part="5"
+F 0 "K11" H 3200 2750 50  0000 C CNN
 F 1 "Genset Power Selected" H 3200 2650 50  0000 C CNN
 F 2 "" H 3850 2500 50  0001 C CNN

Commit message: Updates
Parts:
- D?: symbol device:D_Bridge_+-AA -> power-car-rescue:D_Bridge_+-AA-device
- LA? (x4): symbol device:Lamp -> power-car-rescue:Lamp-device
- T?: symbol device:Transformer_1P_1S -> power-car-rescue:Transformer_1P_1S-device
Changed lines of the file:
@@
 EESchema Schematic File Version 4
 LIBS:power-car-cache
-EELAYER 26 0
+EELAYER 30 0
 EELAYER END
 $Descr USLedger 17000 11000
@@
 Sheet 4 5
 Title ""
-Date "2018-08-05"
-Rev "1.4"
+Date "2019-10-06"
+Rev "1.5"
 Comp ""
 Comment1 ""
@@
 $EndDescr
 $Comp
-L device:Transformer_1P_1S T?
+L power-car-rescue:Transformer_1P_1S-device T?
 U 1 1 5AE7DC6B
 P -7150 6400
@@
 $EndComp
 $Comp
-L device:D_Bridge_+-AA D?
+L power-car-rescue:D_Bridge_+-AA-device D?
 U 1 1 5AE7DE11
 P -6250 6400
@@
 $EndComp
 $Comp
-L device:Lamp LA?
+L power-car-rescue:Lamp-device LA?
 U 1 1 5AF934D7
 P -6550 3300
@@
 $EndComp
 $Comp
-L device:Lamp LA?
+L power-car-rescue:Lamp-device LA?
 U 1 1 5B24EA4F
 P 6350 7350
@@
 $EndComp
 $Comp
-L device:Lamp LA?
+L power-car-rescue:Lamp-device LA?
 U 1 1 5B24EC3A
 P 10500 7650
@@
 $EndComp
 $Comp
-L device:Lamp LA?
+L power-car-rescue:Lamp-device LA?
 U 1 1 5B65C6AB
 P 6200 9600
