File: engine-control.sch (KiCad schematic (older format))
At the start: 26 parts

Commit message: Updates
Parts:
- gave numbers to parts that had none: 8
Connections:
- net Battery_+24V: now also K1.L1; no longer K1.T1
- net Genset_Ctrl_+24V: now also K1.T1; no longer K1.L1
Other:
- note added: "KA-4474-1\n109P198\n24V DC 3CO"
Changed lines of the file:
@@
 EESchema Schematic File Version 4
 LIBS:power-car-cache
-EELAYER 26 0
+EELAYER 30 0
 EELAYER END
 $Descr USLedger 17000 11000
@@
 Sheet 3 5
 Title "Power Car"
-Date "2018-08-05"
-Rev "1.4"
+Date "2019-10-06"
+Rev "1.5"
 Comp "Monticello Railway Museum"
 Comment1 ""
@@
 Genset_Ctrl_+24V
 $Comp
-L mrm:Relay_Octal_11pin_separate K?
+L mrm:Relay_Octal_11pin_separate K5
 U 1 1 5AFE65B3
 P 4100 5100
-AR Path="/5B1A0A6E/5AFE65B3" Ref="K?"  Part="1"
+AR Path="/5B1A0A6E/5AFE65B3" Ref="K5"  Part="1"
 AR Path="/5AE8F0EF/5AFE65B3" Ref="K?"  Part="1"
-F 0 "K?" H 4100 5400 50  0000 C CNN
+F 0 "K5" H 4100 5400 50  0000 C CNN
 F 1 "Low Engine Temp" H 4100 5300 50  0000 C CNN
 F 2 "" H 4500 5150 50  0001 C CNN
@@
 Connection ~ 12950 17700
 $Comp
-L Switch:SW_Push_Dual SW?
+L Switch:SW_Push_Dual SW1
 U 1 1 5B396029
 P 10100 3900
-AR Path="/5B1A0A6E/5B396029" Ref="SW?"  Part="1"
+AR Path="/5B1A0A6E/5B396029" Ref="SW1"  Part="1"
 AR Path="/5AE8F0EF/5B396029" Ref="SW?"  Part="1"
-F 0 "SW?" H 10100 4185 50  0000 C CNN
+F 0 "SW1" H 10100 4185 50  0000 C CNN
 F 1 "Genset Start" H 10100 4094 50  0000 C CNN
 F 2 "" H 10100 4100 50  0001 C CNN
@@
 $EndComp
 $Comp
-L mrm:Relay_Timer K?
+L mrm:Relay_Timer K2
 U 1 1 5B396030
 P 12100 4350
-AR Path="/5B1A0A6E/5B396030" Ref="K?"  Part="1"
+AR Path="/5B1A0A6E/5B396030" Ref="K2"  Part="1"
 AR Path="/5AE8F0EF/5B396030" Ref="K?"  Part="1"
-F 0 "K?" V 11183 4350 50  0000 C CNN
+F 0 "K2" V 11183 4350 50  0000 C CNN
 F 1 "Control Power Timer Relay" V 11274 4350 50  0000 C CNN
 F 2 "" H 12550 4400 50  0001 C CNN
@@
 $EndComp
 $Comp
-L Switch:SW_Push SW?
+L Switch:SW_Push SW2
 U 1 1 5B39604F
 P 10100 5350
-AR Path="/5B1A0A6E/5B39604F" Ref="SW?"  Part="1"
+AR Path="/5B1A0A6E/5B39604F" Ref="SW2"  Part="1"
 AR Path="/5AE8F0EF/5B39604F" Ref="SW?"  Part="1"
-F 0 "SW?" H 10100 5650 50  0000 C CNN
+F 0 "SW2" H 10100 5650 50  0000 C CNN
 F 1 "Genset Stop" H 10100 5550 50  0000 C CNN
 F 2 "" H 10100 5550 50  0001 C CNN
@@
 	11450 4450 11450 4550
 $Comp
-L mrm:Relay_Octal_11pin K?
+L mrm:Relay_Octal_11pin K3
 U 1 1 5B39607D
 P 12100 6900
-AR Path="/5B1A0A6E/5B39607D" Ref="K?"  Part="1"
+AR Path="/5B1A0A6E/5B39607D" Ref="K3"  Part="1"
 AR Path="/5AE8F0EF/5B39607D" Ref="K?"  Part="1"
-F 0 "K?" V 11133 6900 50  0000 C CNN
+F 0 "K3" V 11133 6900 50  0000 C CNN
 F 1 "Genset Remote Run Relay" V 11224 6900 50  0000 C CNN
 F 2 "" H 12450 6950 50  0001 C CNN
@@
 	11200 6500 12500 6500
 $Comp
-L mrm:Contactor_3phase_2NC_2NO K?
+L mrm:Contactor_3phase_2NC_2NO K1
 U 1 1 5B396085
 P 14200 3850
-AR Path="/5B1A0A6E/5B396085" Ref="K?"  Part="1"
+AR Path="/5B1A0A6E/5B396085" Ref="K1"  Part="1"
 AR Path="/5AE8F0EF/5B396085" Ref="K?"  Part="1"
-F 0 "K?" H 14200 4250 50  0000 C CNN
+F 0 "K1" H 14200 4250 50  0000 C CNN
 F 1 "Control Power Contactor" H 14200 4150 50  0000 C CNN
 F 2 "" H 14850 3850 50  0001 C CNN
@@
 $EndComp
 $Comp
-L mrm:Contactor_3phase_2NC_2NO K?
+L mrm:Contactor_3phase_2NC_2NO K1
 U 2 1 5B39608C
 P 14200 4350
-AR Path="/5B1A0A6E/5B39608C" Ref="K?"  Part="2"
+AR Path="/5B1A0A6E/5B39608C" Ref="K1"  Part="2"
 AR Path="/5AE8F0EF/5B39608C" Ref="K?"  Part="2"
-F 0 "K?" H 14200 4505 50  0001 C CNN
+F 0 "K1" H 14200 4505 50  0001 C CNN
 F 1 "Contactor_3phase_2NC_2NO" H 14200 4150 50  0001 C CNN
 F 2 "" H 14850 4350 50  0001 C CNN
 F 3 "" H 14850 4350 50  0001 C CNN
 	2    14200 4350
-	1    0    0    -1
+	-1   0    0    -1
 $EndComp
 Wire Notes Line width 10
@@
 	10300 4100 11200 4100
 $Comp
-L mrm:Relay_Timer K?
+L mrm:Relay_Timer K4
 U 1 1 5B3ADBF7
 P 14050 6000
-AR Path="/5B1A0A6E/5B3ADBF7" Ref="K?"  Part="1"
+AR Path="/5B1A0A6E/5B3ADBF7" Ref="K4"  Part="1"
 AR Path="/5AE8F0EF/5B3ADBF7" Ref="K?"  Part="1"
-F 0 "K?" V 13133 6000 50  0000 C CNN
+F 0 "K4" V 13133 6000 50  0000 C CNN
 F 1 "Cool-down Timer Relay" V 13224 6000 50  0000 C CNN
 F 2 "" H 14500 6050 50  0001 C CNN
@@
 	12500 5350 10300 5350
 $Comp
-L mrm:Relay_Octal_11pin_separate K?
+L mrm:Relay_Octal_11pin_separate K5
 U 2 1 5B430CFF
 P 12100 8150
-F 0 "K?" H 12100 7850 50  0000 C CNN
+F 0 "K5" H 12100 7850 50  0000 C CNN
 F 1 "Low Engine Temp" H 12100 7950 50  0000 C CNN
 F 2 "" H 12750 8150 50  0001 C CNN
@@
 	12400 8250 14650 8250
 $Comp
-L mrm:Relay_Octal_11pin_separate K?
+L mrm:Relay_Octal_11pin_separate K6
 U 1 1 5BB5E4CD
 P 10300 7900
-F 0 "K?" H 10300 8192 50  0000 C CNN
+F 0 "K6" H 10300 8192 50  0000 C CNN
 F 1 "Idle Relay" H 10300 8101 50  0000 C CNN
 F 2 "" H 10700 7950 50  0001 C CNN
@@
 $EndComp
 $Comp
-L mrm:Relay_Octal_11pin_separate K?
+L mrm:Relay_Octal_11pin_separate K6
 U 2 1 5BB5E557
 P 10300 8300
-F 0 "K?" H 10300 8625 50  0001 C CNN
+F 0 "K6" H 10300 8625 50  0001 C CNN
 F 1 "Relay_Octal_11pin_separate" H 10300 8534 50  0001 C CNN
 F 2 "" H 10700 8350 50  0001 C CNN
@@
 	14650 7400 14650 8250
 Connection ~ 14650 7400
+Text Notes 10300 6950 0    50   ~ 0
+KA-4474-1\n109P198\n24V DC 3CO
 $EndSCHEMATC

Commit message: Sturf
Parts:
- added J?: Screw_Terminal_01x11, symbol Connector:Screw_Terminal_01x11
- added LA?: Run, symbol Device:Lamp
- added LA?: Alarm, symbol Device:Lamp
- added LA?: Idle, symbol Device:Lamp
- added LA?: Control Power, symbol Device:Lamp
- added SW?: Ctrl Pwr Force Off, symbol Switch:SW_SPST
- added SW?: Alarm Reset, symbol Switch:SW_Push
- added SW?: EStop, symbol Switch:SW_Push
- added SW? (x2): EStop, symbol Switch:SW_Push_Open
- SW?: value Control Power Enable Override -> Ctrl Pwr Force On
- renumbered K4 to K3, K3 to K4
Connections:
- net GND: now also LA?.1 (-), LA?.1 (-), LA?.1 (-), SW?.1, SW?.1, SW?.1 (A); no longer K4.1
- net Genset_Alarm: now also LA?.2 (+)
- net Genset_Alarm_Reset: now also SW?.2
- net Genset_Ctrl_+24V: now also SW?.1 (A), LA?.1 (-), LA?.2 (+), SW?.2 (B); no longer K3.10 (PWR+), K5.2
- net Idle_Call: now also J?.7 (Pin_7)
- net Idle_Return: now also J?.10 (Pin_10)
- net G8: now reaches SW?.1, SW?.1, SW?.1, TB2.16 (Pin_16)
- net at K5.10: now also SW?.2 (B); no longer SW?.1 (A)
- net G5: now reaches TB2.13 (Pin_13)
- net G5: now also K5.2; no longer SW?.2 (B)
- net at K2.3, SW1.2, SW?.2 (B): now also SW?.1 (A); no longer K1.A1
- net at K2.6 (~START), K3.7 (~RESET), K4.2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: now also LA?.2 (+)
- net at K4.11, K5.1, K6.10: now also LA?.2 (+)
- new net: K4.1, SW?.2 (B)
- new net: K1.A1, SW?.2 (B)
- new net: K3.10 (PWR+), SW?.1 (A)
- new net Genset_Shutdown: SW?.2
Other:
- note added: "Actuator +"
- note added: "Actuator -"
- note added: "Battery +"
- note added: "Battery -"
- note added: "Cabinet"
- note added: "Common"
- note added: "Genset Speed Controller"
- note added: "Idle"
- note added: "Illuminated 3-way switch"
- note added: "Mag Pickup +"
- note added: "Mag Pickup -"
- note added: "Panel"
- note added: "Remote Speed Common"
- note added: "Remote Speed High"
- note added: "Remote Speed Wiper"
- moved on the sheet: CB?, K5A, SW1, SW2, SW?
