File: hep-selection.sch (KiCad schematic (older format))
At the start: 27 parts, among them K1 240V ecoil 750A, K2 240V coil 60A, K3 240V coil 60A, K4 240V ecoil 750A, SW1 HEP Safety Keyswitch, SW2 HEP Dropout, SW3 HEP Pickup

Commit message: Updoots
Parts:
- added CT1, CT2, CT3: Current_Transformer, symbol mrm:Current_Transformer
Connections:
- net labels added: B1, B10, B11, B12, B13, B14, B15, B16, B17, B18, B19, B2, B21, B3, B4, B5, B6, B7, B8, B9
- wire segments 195 -> 201
Other:
- note added: "Place current transformers between\ncurrent source and sinks"
- moved on the sheet: CB?, K2F, K2G, K3G, K?F, SW3

Commit message: more updoots
Parts:
- gave numbers to parts that had none: 2
- renumbered K1 to K11, K2 to K12, K3 to K13, K4 to K14
Connections:
- net labels added: H1, H10, H2, H3, H4, H5, H6, H7, H8, H9
Changed lines of the file:
@@
 $EndComp
 $Comp
-L mrm:Contactor_3phase_2NC_2NO_Eaton_ECoil K1
+L mrm:Contactor_3phase_2NC_2NO_Eaton_ECoil K11
 U 1 1 5ACE6050
 P 5300 2950
-F 0 "K1" H 5300 2700 50  0000 C CNN
+F 0 "K11" H 5300 2700 50  0000 C CNN
 F 1 "240V ecoil 750A" H 5300 2600 50  0000 C CNN
 F 2 "" H 5950 2950 50  0001 C CNN
@@
 $EndComp
 $Comp
-L mrm:Contactor_3phase_2NC_2NO K1
+L mrm:Contactor_3phase_2NC_2NO K11
 U 4 1 5ACE609E
 P 5300 2100
-F 0 "K1" H 5300 2300 50  0001 C CNN
+F 0 "K11" H 5300 2300 50  0001 C CNN
 F 1 "Contactor_3phase_2NC_2NO" H 5300 1900 50  0001 C CNN
 F 2 "" H 5950 2100 50  0001 C CNN
@@
 $EndComp
 $Comp
-L mrm:Contactor_3phase_2NC_2NO K1
+L mrm:Contactor_3phase_2NC_2NO K11
 U 3 1 5ACE60B1
 P 5300 1900
-F 0 "K1" H 5300 2100 50  0001 C CNN
+F 0 "K11" H 5300 2100 50  0001 C CNN
 F 1 "Contactor_3phase_2NC_2NO" H 5300 1700 50  0001 C CNN
 F 2 "" H 5950 1900 50  0001 C CNN
@@
 $EndComp
 $Comp
-L mrm:Contactor_3phase_2NC_2NO K1
+L mrm:Contactor_3phase_2NC_2NO K11
 U 2 1 5ACE60C4
 P 5300 1700
-F 0 "K1" H 5300 1900 50  0001 C CNN
+F 0 "K11" H 5300 1900 50  0001 C CNN
 F 1 "Contactor_3phase_2NC_2NO" H 5300 1500 50  0001 C CNN
 F 2 "" H 5950 1700 50  0001 C CNN
@@
 $EndComp
 $Comp
-L mrm:Contactor_3phase_2NC_2NO K2
+L mrm:Contactor_3phase_2NC_2NO K12
 U 1 1 5ACE6A00
 P 5300 4450
-F 0 "K2" H 5300 4250 50  0000 C CNN
+F 0 "K12" H 5300 4250 50  0000 C CNN
 F 1 "240V coil 60A" H 5300 4150 50  0000 C CNN
 F 2 "" H 5950 4450 50  0001 C CNN
@@
 $EndComp
 $Comp
-L mrm:Contactor_3phase_2NC_2NO K2
+L mrm:Contactor_3phase_2NC_2NO K12
 U 4 1 5ACE6A06
 P 5300 4000
-F 0 "K2" H 5300 4200 50  0001 C CNN
+F 0 "K12" H 5300 4200 50  0001 C CNN
 F 1 "Contactor_3phase_2NC_2NO" H 5300 3800 50  0001 C CNN
 F 2 "" H 5950 4000 50  0001 C CNN
@@
 $EndComp
 $Comp
-L mrm:Contactor_3phase_2NC_2NO K2
+L mrm:Contactor_3phase_2NC_2NO K12
 U 3 1 5ACE6A0C
 P 5300 3800
-F 0 "K2" H 5300 4000 50  0001 C CNN
+F 0 "K12" H 5300 4000 50  0001 C CNN
 F 1 "Contactor_3phase_2NC_2NO" H 5300 3600 50  0001 C CNN
 F 2 "" H 5950 3800 50  0001 C CNN
@@
 $EndComp
 $Comp
-L mrm:Contactor_3phase_2NC_2NO K2
+L mrm:Contactor_3phase_2NC_2NO K12
 U 2 1 5ACE6A12
 P 5300 3600
-F 0 "K2" H 5300 3800 50  0001 C CNN
+F 0 "K12" H 5300 3800 50  0001 C CNN
 F 1 "Contactor_3phase_2NC_2NO" H 5300 3400 50  0001 C CNN
 F 2 "" H 5950 3600 50  0001 C CNN
@@
 $EndComp
 $Comp
-L mrm:Contactor_3phase_2NC_2NO K3
+L mrm:Contactor_3phase_2NC_2NO K13
 U 1 1 5ACE6F6E
 P 5300 6750
-F 0 "K3" H 5300 6550 50  0000 C CNN
+F 0 "K13" H 5300 6550 50  0000 C CNN
 F 1 "240V coil 60A" H 5300 6450 50  0000 C CNN
 F 2 "" H 5950 6750 50  0001 C CNN
@@
 $EndComp
 $Comp
-L mrm:Contactor_3phase_2NC_2NO K3
+L mrm:Contactor_3phase_2NC_2NO K13
 U 4 1 5ACE6F74
 P 5300 6300
-F 0 "K3" H 5300 6500 50  0001 C CNN
+F 0 "K13" H 5300 6500 50  0001 C CNN
 F 1 "Contactor_3phase_2NC_2NO" H 5300 6100 50  0001 C CNN
 F 2 "" H 5950 6300 50  0001 C CNN
@@
 $EndComp
 $Comp
-L mrm:Contactor_3phase_2NC_2NO K3
+L mrm:Contactor_3phase_2NC_2NO K13
 U 3 1 5ACE6F7A
 P 5300 6100
-F 0 "K3" H 5300 6300 50  0001 C CNN
+F 0 "K13" H 5300 6300 50  0001 C CNN
 F 1 "Contactor_3phase_2NC_2NO" H 5300 5900 50  0001 C CNN
 F 2 "" H 5950 6100 50  0001 C CNN
@@
 $EndComp
 $Comp
-L mrm:Contactor_3phase_2NC_2NO K3
+L mrm:Contactor_3phase_2NC_2NO K13
 U 2 1 5ACE6F80
 P 5300 5900
-F 0 "K3" H 5300 6100 50  0001 C CNN
+F 0 "K13" H 5300 6100 50  0001 C CNN
 F 1 "Contactor_3phase_2NC_2NO" H 5300 5700 50  0001 C CNN
 F 2 "" H 5950 5900 50  0001 C CNN
@@
 $EndComp
 $Comp
-L mrm:Contactor_3phase_2NC_2NO K2
+L mrm:Contactor_3phase_2NC_2NO K12
 U 6 1 5ACE91D4
 P 3550 2500
-F 0 "K2" H 3550 2587 50  0000 C CNN
+F 0 "K12" H 3550 2587 50  0000 C CNN
 F 1 "Contactor_3phase_2NC_2NO" H 3550 2300 50  0001 C CNN
 F 2 "" H 4200 2500 50  0001 C CNN
@@
 $EndComp
 $Comp
-L mrm:Contactor_3phase_2NC_2NO K3
+L mrm:Contactor_3phase_2NC_2NO K13
 U 6 1 5ACE9248
 P 4600 2500
-F 0 "K3" H 4600 2587 50  0000 C CNN
+F 0 "K13" H 4600 2587 50  0000 C CNN
 F 1 "Contactor_3phase_2NC_2NO" H 4600 2300 50  0001 C CNN
 F 2 "" H 5250 2500 50  0001 C CNN
@@
 	5600 6300 6300 6300
 $Comp
-L mrm:Contactor_3phase_2NC_2NO K3
+L mrm:Contactor_3phase_2NC_2NO K13
 U 7 1 5ACF90A4
 P 4550 4450
-F 0 "K3" H 4550 4537 50  0000 C CNN
+F 0 "K13" H 4550 4537 50  0000 C CNN
 F 1 "Contactor_3phase_2NC_2NO" H 4550 4250 50  0001 C CNN
 F 2 "" H 5200 4450 50  0001 C CNN
@@
 $EndComp
 $Comp
-L mrm:Contactor_3phase_2NC_2NO K1
+L mrm:Contactor_3phase_2NC_2NO K11
 U 6 1 5ACF9122
 P 3900 4450
-F 0 "K1" H 3900 4537 50  0000 C CNN
+F 0 "K11" H 3900 4537 50  0000 C CNN
 F 1 "Contactor_3phase_2NC_2NO" H 3900 4250 50  0001 C CNN
 F 2 "" H 4550 4450 50  0001 C CNN
@@
 	4200 4450 4250 4450
 $Comp
-L mrm:Contactor_3phase_2NC_2NO K2
+L mrm:Contactor_3phase_2NC_2NO K12
 U 7 1 5AD0C060
 P 3800 6750
-F 0 "K2" H 3800 6837 50  0000 C CNN
+F 0 "K12" H 3800 6837 50  0000 C CNN
 F 1 "Contactor_3phase_2NC_2NO" H 3800 6550 50  0001 C CNN
 F 2 "" H 4450 6750 50  0001 C CNN
@@
 $EndComp
 $Comp
-L mrm:Contactor_3phase_2NC_2NO K1
+L mrm:Contactor_3phase_2NC_2NO K11
 U 7 1 5AD0C066
 P 4600 6750
-F 0 "K1" H 4600 6837 50  0000 C CNN
+F 0 "K11" H 4600 6837 50  0000 C CNN
 F 1 "Contactor_3phase_2NC_2NO" H 4600 6550 50  0001 C CNN
 F 2 "" H 5250 6750 50  0001 C CNN
@@
 	3350 6750 3500 6750
 $Comp
-L mrm:Contactor_3phase_2NC_2NO K4
+L mrm:Contactor_3phase_2NC_2NO K14
 U 2 1 5AD96CCE
 P 5300 7600
-F 0 "K4" H 5300 7850 50  0000 C CNN
+F 0 "K14" H 5300 7850 50  0000 C CNN
 F 1 "240V ecoil 750A" H 5300 7750 50  0000 C CNN
 F 2 "" H 5950 7600 50  0001 C CNN
@@
 $EndComp
 $Comp
-L mrm:Contactor_3phase_2NC_2NO K?
+L mrm:Contactor_3phase_2NC_2NO K14
 U 3 1 5AD96D1A
 P 5300 7800
-F 0 "K?" H 5300 8000 50  0001 C CNN
+F 0 "K14" H 5300 8000 50  0001 C CNN
 F 1 "Contactor_3phase_2NC_2NO" H 5300 7600 50  0001 C CNN
 F 2 "" H 5950 7800 50  0001 C CNN
@@
 $EndComp
 $Comp
-L mrm:Contactor_3phase_2NC_2NO K?
+L mrm:Contactor_3phase_2NC_2NO K14
 U 4 1 5AD96D3D
 P 5300 8000
-F 0 "K?" H 5300 8200 50  0001 C CNN
+F 0 "K14" H 5300 8200 50  0001 C CNN
 F 1 "Contactor_3phase_2NC_2NO" H 5300 7800 50  0001 C CNN
 F 2 "" H 5950 8000 50  0001 C CNN
@@
 $EndComp
 $Comp
-L mrm:Contactor_3phase_2NC_2NO K2
+L mrm:Contactor_3phase_2NC_2NO K12
 U 5 1 5ADC4A44
 P 8300 5700
-F 0 "K2" H 8300 5950 50  0000 C CNN
+F 0 "K12" H 8300 5950 50  0000 C CNN
 F 1 "Standby Power Selected" H 8300 5850 50  0000 C CNN
 F 2 "" H 8950 5700 50  0001 C CNN
@@
 $EndComp
 $Comp
-L mrm:Contactor_3phase_2NC_2NO K1
+L mrm:Contactor_3phase_2NC_2NO K11
 U 5 1 5ADC7F52
 P 8300 5300
-F 0 "K1" H 8300 5550 50  0000 C CNN
+F 0 "K11" H 8300 5550 50  0000 C CNN
 F 1 "Genset Power Selected" H 8300 5450 50  0000 C CNN
 F 2 "" H 8950 5300 50  0001 C CNN
@@
 	12300 8400 12500 8400
 $Comp
-L mrm:Contactor_3phase_2NC_2NO_Eaton_ECoil K4
+L mrm:Contactor_3phase_2NC_2NO_Eaton_ECoil K14
 U 1 1 5AEAABC4
 P 13500 7500
-F 0 "K4" H 13500 8050 50  0000 C CNN
+F 0 "K14" H 13500 8050 50  0000 C CNN
 F 1 "240V ecoil 750A" H 13500 7950 50  0000 C CNN
 F 2 "" H 14150 7500 50  0001 C CNN
@@
 $EndComp
 $Comp
-L mrm:Contactor_3phase_2NC_2NO K4
+L mrm:Contactor_3phase_2NC_2NO K14
 U 5 1 5AEB0464
 P 13500 8150
-F 0 "K4" H 13500 7950 50  0001 C CNN
+F 0 "K14" H 13500 7950 50  0001 C CNN
 F 1 "24V coil 350A" H 13500 8350 50  0001 C CNN
 F 2 "" H 14150 8150 50  0001 C CNN
@@
 NoConn ~ 13800 7650
 $Comp
-L mrm:Contactor_3phase_2NC_2NO K?
+L mrm:Contactor_3phase_2NC_2NO K14
 U 8 1 5B077E99
 P 13500 8400
-F 0 "K?" H 13500 8200 50  0001 C CNN
+F 0 "K14" H 13500 8200 50  0001 C CNN
 F 1 "Contactor_3phase_2NC_2NO" H 13500 8600 50  0001 C CNN
 F 2 "" H 14150 8400 50  0001 C CNN
@@
 	4650 7800 5000 7800
 $Comp
-L mrm:Contactor_3phase_2NC_2NO K?
+L mrm:Contactor_3phase_2NC_2NO K15
 U 1 1 5AEBB9BB
 P 4200 8700
-F 0 "K?" H 4200 8900 50  0000 C CNN
+F 0 "K15" H 4200 8900 50  0000 C CNN
 F 1 "HEP Voltage Detect" H 4200 8500 50  0000 C CNN
 F 2 "" H 4850 8700 50  0001 C CNN
@@
 $EndComp
 $Comp
-L mrm:Contactor_3phase_2NC_2NO K?
+L mrm:Contactor_3phase_2NC_2NO K15
 U 6 1 5AEBBAA6
 P 12700 7850
-F 0 "K?" H 12700 7950 50  0000 C CNN
+F 0 "K15" H 12700 7950 50  0000 C CNN
 F 1 "HEP Voltage Detect" H 12700 7750 50  0000 C CNN
 F 2 "" H 13350 7850 50  0001 C CNN
@@
 B15
 Text Label 6550 2800 0    50   ~ 0
-B1
+B9
 Text Label 6750 2800 0    50   ~ 0
-B2
+B10
 Text Label 6950 2800 0    50   ~ 0
-B3
+B11
 Text Label 7150 2800 0    50   ~ 0
-B4
+B12
 Text Label 7350 2800 0    50   ~ 0
-B5
+B13
 Text Label 7550 2800 0    50   ~ 0
-B6
+B14
 Text Label 13850 8400 0    50   ~ 0
 B16
 Wire Notes Line
-	12900 8250 12900 8550
-Wire Notes Line
-	12900 8550 14150 8550
+	13050 8250 13050 8550
+Wire Notes Line
+	13050 8550 14150 8550
 Wire Notes Line
 	14150 6850 14150 8550
 Wire Notes Line
-	12900 8250 11400 8250
+	13050 8250 11400 8250
 Wire Notes Line
 	7700 5400 7700 4950
@@
 	14000 8575 13975 8550
 Text Label 3050 2250 0    50   ~ 0
-B7
+B1
 Wire Wire Line
 	1900 2700 5000 2700
@@
 	3850 2500 4300 2500
 Text Label 4000 2500 0    50   ~ 0
-B8
+B2
 Wire Notes Line
 	3950 2300 3950 3450
@@
 	3950 3450 5800 3450
 Text Label 4000 2700 0    50   ~ 0
-B9
+B3
 Text Label 4000 2800 0    50   ~ 0
-B10
+B4
 Text Label 3550 4450 1    50   ~ 0
-B11
+B5
 Connection ~ 4250 4450
 Wire Wire Line
@@
 	4850 4450 5000 4450
 Text Label 4950 4450 1    50   ~ 0
-B12
+B6
 Text Label 3500 5250 0    50   ~ 0
-B13
+B7
 Connection ~ 3500 6750
 Wire Wire Line
@@
 	4100 6750 4300 6750
 Text Label 4250 6750 1    50   ~ 0
-B14
+B8
 Text Label 8800 5300 2    50   ~ 0
 B17
@@
 Text Label 13950 7250 0    50   ~ 0
 B21
+Text Label 9750 5700 1    50   ~ 0
+H1
+Text Label 10250 5700 1    50   ~ 0
+H2
+Text Label 10400 5700 1    50   ~ 0
+H7
+Text Label 10400 6100 1    50   ~ 0
+H8
+Text Label 9750 6100 1    50   ~ 0
+H5
+Text Label 10250 6100 1    50   ~ 0
+H6
+Text Label 8050 6100 1    50   ~ 0
+H3
+Text Label 9200 6100 1    50   ~ 0
+H4
+Text Label 11950 8400 1    50   ~ 0
+H10
+Text Label 13000 8400 1    50   ~ 0
+H9
 $EndSCHEMATC

Commit message: Updates
Parts:
- C1: symbol device:CP1 -> power-car-rescue:CP1-device
- D1, D3, D4: symbol device:LED -> power-car-rescue:LED-device
- D?: symbol device:D_Bridge_+-AA -> power-car-rescue:D_Bridge_+-AA-device
- R1, R3, R4: symbol device:R -> power-car-rescue:R-device
- T? (x2): symbol device:Transformer_1P_1S -> power-car-rescue:Transformer_1P_1S-device
Changed lines of the file:
@@
 EESchema Schematic File Version 4
 LIBS:power-car-cache
-EELAYER 26 0
+EELAYER 30 0
 EELAYER END
 $Descr USLedger 17000 11000
@@
 Sheet 2 5
 Title "Power Car"
-Date "2018-08-05"
-Rev "1.4"
+Date "2019-10-06"
+Rev "1.5"
 Comp "Monticello Railway Museum"
 Comment1 ""
@@
 	11800 3100 11700 3100
 $Comp
-L device:Transformer_1P_1S T?
+L power-car-rescue:Transformer_1P_1S-device T?
 U 1 1 5AD7B1F0
 P 12200 3300
@@
 	10600 2400 10400 2400
 $Comp
-L device:Transformer_1P_1S T?
+L power-car-rescue:Transformer_1P_1S-device T?
 U 1 1 5AD714B0
 P 11000 2600
@@
 Trainline Safety Loop
 $Comp
-L device:R R1
+L power-car-rescue:R-device R1
 U 1 1 5ADE2274
 P 8850 6100
@@
 $EndComp
 $Comp
-L device:LED D1
+L power-car-rescue:LED-device D1
 U 1 1 5ADE24E4
 P 8350 6100
@@
 $EndComp
 $Comp
-L device:R R4
+L power-car-rescue:R-device R4
 U 1 1 5AE78376
 P 12150 8400
@@
 $EndComp
 $Comp
-L device:LED D4
+L power-car-rescue:LED-device D4
 U 1 1 5AE7837D
 P 12650 8400
@@
 Local_110V_L2
 $Comp
-L device:D_Bridge_+-AA D?
+L power-car-rescue:D_Bridge_+-AA-device D?
 U 1 1 5B1FDD26
 P 13650 3300
@@
 	12900 3600 13650 3600
 $Comp
-L device:R R3
+L power-car-rescue:R-device R3
 U 1 1 5B244082
 P 13900 4300
@@
 $EndComp
 $Comp
-L device:LED D3
+L power-car-rescue:LED-device D3
 U 1 1 5B244088
 P 13400 4300
@@
 	14150 3300 14150 3900
 $Comp
-L device:CP1 C1
+L power-car-rescue:CP1-device C1
 U 1 1 5B3013F7
 P 13600 3900

Commit message: Sturf
Connections:
- wire segments 201 -> 202
Other:
- moved on the sheet: D1, D4, K11E, K12E, K14A, K15F, K?, K?C, R1, R4, SW1, SW2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
